File: SetSeg.kicad_sch (KiCad schematic)
At the start: 19 parts, among them U4 74AHC04, U5 74AHC04, U6 D148K, U7 74AHC04, U8 D148K

Commit message: Atualizados os Footprints. Definido um primeiro corte da placa.
Parts:
- R17, R18, R19, R20, R21, R22, R23, R24, R25, R26, R27, R28, R29, R30: footprint Resistor_THT:R_Axial_DIN0204_L3.6mm_D1.6mm_P5.08mm_Horizontal -> Resistor_THT:R_Axial_DIN0207_L6.3mm_D2.5mm_P7.62mm_Horizontal
- U4, U5, U7: footprint Package_DIP:DIP-14_W7.62mm_Socket -> Package_DIP:DIP-14_W7.62mm

Commit message: Placa roeada automaticamente.
Parts:
- added C4, C5: 10uF, Capacitor_THT:CP_Radial_D5.0mm_P2.50mm, symbol Device:C_Polarized
- added unit 7 of U4
- added unit 7 of U5
- renumbered U4 to U3, U5 to U4, U7 to U5
Connections:
- net GND: now also C4.2, C5.2, U4.7 (GND), U5.7 (GND)
- new net +5V: C4.1, C5.1, U4.14 (VCC), U5.14 (VCC)
Other:
- company: (none) -> IFTM - Campus Ituiutaba
- title: (none) -> FPGA LED Output Board - 7 Segment Display
